File: Hydroponics Shield/Hydroponics Shield Rev2/hydroponics_shield_rev2.kicad_pcb (KiCad board)
At the start: 2 copper layers, 142.2 x 69.1 mm, 83 parts, among them CON1 PJ-202A, J1 282836-6, J2 282836-6, P1 CONN_01X07, P2 0022053031, P4 22-05-3021, P5 22-05-3021, P9 0731000105, Q1 DMN65D8L-7, Q5 PSMN022-30PL,127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

Commit message: update
Parts:
- removed P1: CONN_01X07, Pin_Headers:Pin_Header_Angled_1x07
- removed R1, R2, R3: 10.0k, Resistors_SMD:R_0805_HandSoldering
- added J3: RJHSE-5080, USER_CONNECTORS:RJHSE-5080, F.Cu at (50.8, 61.0)
- added JP1: Jumper_NO_Small, Pin_Headers:Pin_Header_Straight_1x02, F.Cu at (23.6, 71.9)
- added P3: MTG, Mounting_Holes:MountingHole_2-7mm, F.Cu at (24.4, 122.4)
- added P6: MTG, Mounting_Holes:MountingHole_2-7mm, F.Cu at (24.4, 91.9)
- added P7: MTG, Mounting_Holes:MountingHole_2-7mm, F.Cu at (160.3, 122.4)
- added P8: MTG, Mounting_Holes:MountingHole_2-7mm, F.Cu at (160.3, 72.9)
- moved P2 17.8 mm to (70.1, 68.1)
- moved R6 1.83 mm to (28.4, 108.2), turned to 90 degrees
Connections:
- P2 pad 1: GND -> +5V
- P2 pad 3: +5V -> GND
- R4 pad 2: +5V -> +3V3
- R5 pad 2: +5V -> +3V3
- SHIELD1 pad 13: Net-(SHIELD1-Pad13) -> DISPLAY_RESET
Routing:
- net GND: track 109.2 -> 57.8 mm, vias 10 -> 9
- net DISPLAY_RESET: track 0.00 -> 47.8 mm, vias 0 -> 2
- net +3V3: track 87.6 -> 124.6 mm, vias 0 -> 2
- net TEMP_SENSE_IN: track 61.2 -> 75.8 mm, vias 4 -> 2
- net ENCODER_A: track 55.3 -> 65.0 mm, vias 1 -> 2
- net ENCODER_B: track 52.7 -> 62.2 mm, vias 1 -> 2
- net ENCODER_SW: track 50.5 -> 59.4 mm, vias 1 -> 2
- net +5V: track 226.2 -> 234.6 mm, vias 5 -> 6
- net +12V: track 282.2 -> 273.8 mm
- net SCL: track 118.5 -> 125.4 mm, vias 5 -> 4
- net Vguard: track 47.5 -> 53.7 mm
- net FLOAT_SWITCH_IN: track 56.1 -> 60.2 mm, vias 2 -> 3
- net Net-(JP1-Pad1): track 3.84 -> 7.38 mm
- net SDA: track 120.9 -> 118.0 mm, vias 3 -> 6
- net PH_VOUT: track 36.3 -> 34.8 mm
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
Commit message: .
Parts:
- added BAT1: BS-7_2032, USER_CONNECTORS:BS-7_USER, B.Cu at (115.3, 104.6)
- added D1: 1N4448W-TP, Diodes_SMD:SOD-123, F.Cu at (50.5, 82.5)
- added D6: 1N4448W-TP, Diodes_SMD:SOD-123, F.Cu at (51.1, 86.0)
- R12: value 10.0k -> 0
- R13: value 10.0k -> DNP
- R17, R18: value 10.0k -> 10.0k 0.1%
Connections:
- C8 pad 2: +5V -> Net-(C8-Pad2)
- U2 pad 8: +5V -> Net-(C8-Pad2)
Routing:
- net BATT_BACKUP: track 0.00 -> 87.7 mm, vias 0 -> 2
- net +5V: track 234.6 -> 225.0 mm, vias 6 -> 4
- net Net-(C8-Pad2): track 0.00 -> 6.79 mm
- net GND: track 57.8 -> 61.9 mm, vias 9 -> 12
- net SCL: track 125.4 -> 127.7 mm
- net SDA: track 118.0 -> 116.4 mm, vias 6 -> 4
- net TEMP_SENSE_IN: track 75.8 -> 75.2 mm
- net LED_STRIP_OUT: track 97.2 -> 96.7 mm
- net +12V: track 273.8 -> 274.3 mm
Other:
- board text added: "FLOAT SWITCH"
