File: Hydroponics Shield/Hydroponics Shield Rev2/hydroponics_shield_rev2.kicad_pcb (KiCad board)
At the start: 2 copper layers, 142.2 x 69.1 mm, 88 parts, among them CON1 PJ-202A, J1 282836-6, J2 282836-6, J3 RJHSE-5080, P2 0022053031, P3 MTG, P4 22-05-3021, P5 22-05-3021, P6 MTG, P7 MTG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

Commit message: rev4
Connections:
- net Net-(D14-Pad2) renamed /esptx
- net Net-(PCB1-Pad7) renamed /esprx
- LED1 pad 4: Net-(LED1-Pad4) -> (no net)
- P3 pad 1: Net-(P3-Pad1) -> (no net)
- P6 pad 1: Net-(P6-Pad1) -> (no net)
- P7 pad 1: Net-(P7-Pad1) -> (no net)
- P8 pad 1: Net-(P8-Pad1) -> (no net)
- PCB1 pad 5: Net-(PCB1-Pad5) -> (no net)
- PCB1 pad 6: Net-(PCB1-Pad6) -> (no net)
- REF1 pad 1: Net-(REF1-Pad1) -> (no net)
- SHIELD1 pad 0: Net-(SHIELD1-Pad0) -> (no net)
- SHIELD1 pad 1: Net-(SHIELD1-Pad1) -> (no net)
- SHIELD1 pad 3V3: Net-(SHIELD1-Pad3V3) -> (no net)
- SHIELD1 pad AREF: Net-(SHIELD1-PadAREF) -> (no net)
- SHIELD1 pad IORE: Net-(SHIELD1-PadIORE) -> (no net)
- SHIELD1 pad RST: Net-(SHIELD1-PadRST) -> (no net)
- U2 pad 3: Net-(U2-Pad3) -> (no net)
- U2 pad 7: Net-(U2-Pad7) -> (no net)
