File: Hydroponics Shield/Hydroponics Shield Rev3/hydroponics_shield_rev3.kicad_pcb (KiCad board)
At the start: 2 copper layers, 142.2 x 79.8 mm, 90 parts, among them CON1 PJ-202A, J1 282836-6, J2 282836-6, J3 RJHSE-5080, J5 SJ-2523-SMT-TR, J6 SJ-2523-SMT-TR, P1 CONN_01X02, P3 MTG, P6 MTG, P7 MTG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

Commit message: rev4
Parts:
- moved C16 7.26 mm to (79.0, 68.3), turned to 90 degrees
- moved CON1 1.41 mm to (86.9, 54.4)
Routing:
- net +12V: track 269.1 -> 261.8 mm
- net +5V: track 239.2 -> 234.8 mm
- net GND: track 72.2 -> 71.6 mm
Other:
- rule trace_min: 0.2 -> 0
