File: Hydroponics Shield/Hydroponics Shield Rev3/hydroponics_shield_rev3.sch (KiCad schematic (older format))
At the start: 90 parts, among them CON1 PJ-202A, J1 282836-6, J2 282836-6, J3 RJHSE-5080, J5 SJ-2523-SMT-TR, J6 SJ-2523-SMT-TR, P1 CONN_01X02, P3 MTG, P6 MTG, P7 MTG, P8 MTG, P9 0731000105, Q1 DMN65D8L-7, Q5 PSMN022-30PL,127, Q6 PSMN022-30PL,127, Q7 PSMN022-30PL,127, Q8 PSMN022-30PL,127, Q9 PSMN022-30PL,127, U1 LMC6482IN, U2 PCF8563, U3 AZ1117CH-3_3TRG1, U4 AZ1117CH-5TRG1, U5 ESP32_devkitc, Y1 CFS-20632768DZFB

Commit message: rev4
Parts:
- BAT1: symbol BS-7_2032 -> USER_CONNECTORS:BS-7_2032
- C1, C11, C12, C15, C16, C2, C7, C8, C9: symbol C_Small -> Device:C_Small
- C10, C13, C14, C17: symbol C -> USER_SYMBOLS:C
- C3, C4, C5, C6: symbol 5ZLH100MEFC6.3X11 -> USER_CAPACITORS:5ZLH100MEFC6.3X11
- CON1: symbol BARREL_JACK -> Connector:Barrel_Jack_Switch
- D1, D6: symbol 1N4448W-TP -> USER_DIODES:1N4448W-TP
- D11, D13, D14, D17, D18, D19, D20, D21, D8, D9: symbol Led_Small -> Device:LED_Small
- D2, D3, D4, D5: symbol S1GTR -> USER_DIODES:S1GTR
- J1, J2: symbol 282836-6 -> USER_CONNECTORS:282836-6
- J3: symbol RJHSE-5080 -> USER_CONNECTORS:RJHSE-5080
- J5, J6: symbol SJ-2523-SMT-TR -> USER_CONNECTORS:SJ-2523-SMT-TR
- JP1: symbol Jumper_NO_Small -> Device:Jumper_NO_Small
- LED1: symbol COM-12999(WS2812) -> USER_DIODES:COM-12999(WS2812)
- P1: symbol CONN_01X02 -> Connector_Generic:Conn_01x02
- P3, P6, P7, P8: symbol CONN_01X01 -> OLD_LIBS:CONN_01X01
- P9: symbol 0731000105 -> USER_CONNECTORS:0731000105
- Q1: symbol DMN65D8L-7 -> USER_MOSFETS:DMN65D8L-7
- Q5, Q6, Q7, Q8, Q9: symbol PSMN022-30PL,127 -> USER_MOSFETS:PSMN022-30PL,127
- R10, R11, R12, R13, R14, R15, R16, R17, R18, R20, R21, R22, R26, R27, R29, R31, R32, R35, R36, R37, R38, R39, R4, R5, R6, R7, R8, R9: symbol R -> USER_SYMBOLS:R
- REF1: symbol LT1004CZ-2.5 -> USER_DIODES:LT1004CZ-2.5
- SHIELD1: symbol ARDUINO_SHIELD_R3_WI2C -> USER_MODULES:ARDUINO_SHIELD_R3_WI2C
- U1: symbol LMC6482IN -> USER_OPAMPS:LMC6482IN
- U2: symbol PCF8563 -> USER_MODULES:PCF8563
- U3, U4: symbol AZ1117CH-3_3TRG1 -> dk_PMIC-Voltage_Regulators-Linear:AZ1117CH-3_3TRG1
- U5: symbol ESP32_devkitc -> USER_MODULES:ESP32_devkitc
- Y1: symbol CFS-20632768DZFB -> USER_CLOCKS_CRYSTALS:CFS-20632768DZFB
Connections:
- wire segments 302 -> 388
