File: Controller Board/Controller Board Rev2/controller_board.sch (KiCad schematic (older format))
At the start: 23 parts, among them J1 RJHSE-5080, U1 AZ1117CH-3_3TRG1

Commit message: rev4
Parts:
- R10: value 0 -> DNP]
- R11: value DNP -> 0
Changed lines of the file:
@@
 P 5600 3600
 F 0 "R11" V 5500 3600 50  0000 C CNN
-F 1 "DNP" V 5700 3600 50  0000 C CNN
+F 1 "0" V 5700 3600 50  0000 C CNN
 F 2 "Resistors_SMD:R_0805_HandSoldering" V 5530 3600 30  0001 C CNN
 F 3 "" H 5525 3600 30  0000 C CNN
@@
 P 5600 3200
 F 0 "R10" V 5500 3200 50  0000 C CNN
-F 1 "0" V 5700 3200 50  0000 C CNN
+F 1 "DNP]" V 5700 3200 50  0000 C CNN
 F 2 "Resistors_SMD:R_0805_HandSoldering" V 5530 3200 30  0001 C CNN
 F 3 "" H 5525 3200 30  0000 C CNN

Commit message: Long overdue
Parts:
- C2, C4: symbol C_Small -> controller_board-rescue:C_Small
- C3: symbol 5ZLH100MEFC6.3X11 -> USER_CAPACITORS:5ZLH100MEFC6.3X11
- D1, D2, D3, D4: symbol Led_Small -> controller_board-rescue:Led_Small
- DS1: symbol OLED_GENERIC_SSD1305_20PIN_128x64 -> USER_DISPLAY:OLED_GENERIC_SSD1305_20PIN_128x64
- ENC1: symbol EC11K1524406 -> USER_MECHANICAL_OTHER:EC11K1524406
- J1: symbol RJHSE-5080 -> USER_CONNECTORS:RJHSE-5080
- R1, R10, R11, R12, R2, R3, R4, R5, R6, R7, R8, R9: symbol R -> USER_SYMBOLS:R
- U1: symbol AZ1117CH-3_3TRG1 -> dk_PMIC-Voltage_Regulators-Linear:AZ1117CH-3_3TRG1
